File: lcd-panel/lcd-panel.kicad_sch (KiCad schematic)
At the start: 30 parts, among them J1 USB wire, J2 LCD FPC connector, J3 Fan Socket, Q1 AO3400A, U1 FT232HL-REEL, U2 93LC56BT-I/OT, U3 USBLC6-2SC6, Y1 12 MHz, 20 pF load

Commit message: Swapping the LCD socket to the top connectors one
Parts:
- J2: LCSC C506791 -> C324723
Changed lines of the file:
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@@
 			)
 		)
-		(property "LCSC" "C506791"
+		(property "LCSC" " C324723"
 			(at 242.57 50.8 0)
 			(effects
