File: lcd-panel/lcd-panel.kicad_sch (KiCad schematic)
At the start: 46 parts, among them J1 USB wire, J2 LCD FPC connector, J3 Fan Socket, J4 TC2030, Q1 AO3400A, Q2 AO3401A, Q3 AO3400A, U1 FT232HL-REEL, U2 93LC56BT-I/OT, U3 USBLC6-2SC6, U4 ATtiny414-SS, Y1 12 MHz, 20 pF load

Commit message: Spit and polish
Parts:
- J2: LCSC C324723 -> C5139870
Changed lines of the file:
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@@
 			)
 		)
-		(property "LCSC" " C324723"
+		(property "LCSC" " C5139870"
 			(at 266.7 38.1 0)
 			(effects
